Commit message: urdf file

File: Robot_Model_Description/urdf/Robot_Model_Description.urdf (robot description, URDF)
Before this commit: robot my_robot_description, 5 links, 4 joints
Links:
- removed link left_back_wheel_link
- removed link left_front_wheel_link
- removed link right_back_wheel_link
- removed link right_front_wheel_link
- added link BackLeft_Wheel_Link, mass 0.0969966731795848; collision mesh filename=package://Robot_Model_Description/meshes/BackLeft_Wheel_Lin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; visual mesh filename=package://Robot_Model_Description/meshes/BackLeft_Wheel_Lin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
- added link BackRight_Wheel_Link, mass 0.0969966731795849; collision mesh filename=package://Robot_Model_Description/meshes/BackRight_Wheel_Li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; visual mesh filename=package://Robot_Model_Description/meshes/BackRight_Wheel_Li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
- added link FrontLeft_Wheel_Link, mass 0.0969966731795848; collision mesh filename=package://Robot_Model_Description/meshes/FrontLeft_Wheel_Li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; visual mesh filename=package://Robot_Model_Description/meshes/FrontLeft_Wheel_Li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
- added link FrontRight_Wheel_Link, mass 0.0969966731795849; collision mesh filename=package://Robot_Model_Description/meshes/FrontRight_Wheel_L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; visual mesh filename=package://Robot_Model_Description/meshes/FrontRight_Wheel_L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
- link base_link: mass 1.26542477796077 -> 1.29342477796077; geometry collision mesh filename=package://Robot_Model_Description/meshes/base_link.STL; visual mesh filename=package://Robot_Model_Description/meshes/base_link.STL
Joints:
- removed joint left_back_wheel_joint
- removed joint left_front_wheel_joint
- removed joint right_back_wheel_joint
- removed joint right_front_wheel_joint
- added joint BackLeft_Wheel_Joint: type continuous, parent base_link, child BackLeft_Wheel_Link, origin xyz=-0.0079307 -0.16222 0.047088 rpy=1.5708 1.5708 0, axis 0 1 0, limit effort=100 velocity=100
- added joint BackRight_Wheel_Joint: type continuous, parent base_link, child BackRight_Wheel_Link, origin xyz=0.19207 -0.16222 0.047088 rpy=1.5708 -1.5708 0, axis 0 1 0, limit effort=100 velocity=100
- added joint FrontLeft_Wheel_Joint: type continuous, parent base_link, child FrontLeft_Wheel_Link, origin xyz=-0.0079307 -0.16222 0.24709 rpy=1.5708 1.5708 0, axis 0 1 0, limit effort=100 velocity=100
- added joint FrontRight_Wheel_Joint: type continuous, parent base_link, child FrontRight_Wheel_Link, origin xyz=0.19207 -0.16222 0.24709 rpy=1.5708 -1.5708 0, axis 0 1 0, limit effort=100 velocity=100
