Commit message: new urdf update

File: my_robot_description/urdf/my_robot_description.urdf (robot description, URDF)
Before this commit: robot Robot_Model_Description, 5 links, 4 joints
Links:
- removed link BackLeft_Wheel_Link
- removed link BackRight_Wheel_Link
- removed link FrontLeft_Wheel_Link
- removed link FrontRight_Wheel_Link
- added link leftback_wheel_link, mass 0.0969966731795849; collision mesh filename=package://my_robot_description/meshes/leftback_wheel_link.S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; visual mesh filename=package://my_robot_description/meshes/leftback_wheel_link.S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
- added link leftfront_wheel_link, mass 0.0969966731795849; collision mesh filename=package://my_robot_description/meshes/leftfront_wheel_link.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; visual mesh filename=package://my_robot_description/meshes/leftfront_wheel_link.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
- added link rightback_wheel_link, mass 0.0969966731795849; collision mesh filename=package://my_robot_description/meshes/rightback_wheel_link.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; visual mesh filename=package://my_robot_description/meshes/rightback_wheel_link.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
- added link rightfront_wheel_link, mass 0.0969966731795849; collision mesh filename=package://my_robot_description/meshes/rightfront_wheel_link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; visual mesh filename=package://my_robot_description/meshes/rightfront_wheel_link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
- link base_link: mass 1.29342477796077 -> 1.26542477796077; geometry collision mesh filename=package://my_robot_description/meshes/base_link.STL; visual mesh filename=package://my_robot_description/meshes/base_link.STL
Joints:
- removed joint BackLeft_Wheel_Joint
- removed joint BackRight_Wheel_Joint
- removed joint FrontLeft_Wheel_Joint
- removed joint FrontRight_Wheel_Joint
- added joint leftback_wheel_joint: type continuous, parent base_link, child leftback_wheel_link, origin xyz=0 0.115 0.05 rpy=1.5708 1.5708 0, axis 0 1 0, limit effort=100 velocity=100
- added joint leftfront_wheel_joint: type continuous, parent base_link, child leftfront_wheel_link, origin xyz=0 0.115 0.25 rpy=1.5708 1.5708 0, axis 0 1 0, limit effort=100 velocity=100
- added joint rightback_wheel_joint: type continuous, parent base_link, child rightback_wheel_link, origin xyz=0.2 0.115 0.05 rpy=1.5708 -1.5708 0, axis 0 1 0, limit effort=100 velocity=100
- added joint rightfront_wheel_joint: type continuous, parent base_link, child rightfront_wheel_link, origin xyz=0.2 0.115 0.25 rpy=1.5708 -1.5708 0, axis 0 1 0, limit effort=100 velocity=100

Commit message: new robot urdf

File: my_robot_description/urdf/my_robot_description.urdf (robot description, URDF)
Before this commit: robot my_robot_description, 5 links, 4 joints
Links:
- removed link leftback_wheel_link
- removed link leftfront_wheel_link
- removed link rightback_wheel_link
- removed link rightfront_wheel_link
- added link left_back_wheel_link, mass 0.0969966731795849; collision mesh filename=package://my_robot_description/meshes/left_back_wheel_link.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; visual mesh filename=package://my_robot_description/meshes/left_back_wheel_link.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
- added link left_front_wheel_link, mass 0.0969966731795849; collision mesh filename=package://my_robot_description/meshes/left_front_wheel_link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; visual mesh filename=package://my_robot_description/meshes/left_front_wheel_link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
- added link right_back_wheel_link, mass 0.0969966731795849; collision mesh filename=package://my_robot_description/meshes/right_back_wheel_link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; visual mesh filename=package://my_robot_description/meshes/right_back_wheel_link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
- added link right_front_wheel_link, mass 0.0969966731795849; collision mesh filename=package://my_robot_description/meshes/right_front_wheel_lin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; visual mesh filename=package://my_robot_description/meshes/right_front_wheel_lin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
Joints:
- removed joint leftback_wheel_joint
- removed joint leftfront_wheel_joint
- removed joint rightback_wheel_joint
- removed joint rightfront_wheel_joint
- added joint left_back_wheel_joint: type continuous, parent base_link, child left_back_wheel_link, origin xyz=0.2 0.25 -0.115 rpy=1.5708 -1.5708 0, axis 0 1 0, limit effort=100 velocity=100
- added joint left_front_wheel_joint: type continuous, parent base_link, child left_front_wheel_link, origin xyz=0.2 0.05 -0.115 rpy=1.5708 -1.5708 0, axis 0 1 0, limit effort=100 velocity=100
- added joint right_back_wheel_joint: type continuous, parent base_link, child right_back_wheel_link, origin xyz=0 0.25 -0.115 rpy=1.5708 1.5708 0, axis 0 1 0, limit effort=100 velocity=100
- added joint right_front_wheel_joint: type continuous, parent base_link, child right_front_wheel_link, origin xyz=0 0.05 -0.115 rpy=1.5708 1.5708 0, axis 0 1 0, limit effort=100 velocity=100

Commit message: Robot URDF

File: my_robot_description/urdf/my_robot_description.urdf (robot description, URDF)
Before this commit: robot Robot_Model_Description, 5 links, 4 joints
Links:
- removed link BackLeft_Wheel_Link
- removed link BackRight_Wheel_Link
- removed link FrontLeft_Wheel_Link
- removed link FrontRight_Wheel_Link
- added link left_back_wheel_link, mass 0.0969966731795849; collision mesh filename=package://my_robot_description/meshes/left_back_wheel_link.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; visual mesh filename=package://my_robot_description/meshes/left_back_wheel_link.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
- added link left_front_wheel_link, mass 0.0969966731795849; collision mesh filename=package://my_robot_description/meshes/left_front_wheel_link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; visual mesh filename=package://my_robot_description/meshes/left_front_wheel_link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
- added link right_back_wheel_link, mass 0.0969966731795849; collision mesh filename=package://my_robot_description/meshes/right_back_wheel_link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; visual mesh filename=package://my_robot_description/meshes/right_back_wheel_link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
- added link right_front_wheel_link, mass 0.0969966731795849; collision mesh filename=package://my_robot_description/meshes/right_front_wheel_lin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; visual mesh filename=package://my_robot_description/meshes/right_front_wheel_lin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
- link base_link: mass 1.29342477796077 -> 1.45942477796077; geometry collision mesh filename=package://my_robot_description/meshes/base_link.STL; visual mesh filename=package://my_robot_description/meshes/base_link.STL
Joints:
- removed joint BackLeft_Wheel_Joint
- removed joint BackRight_Wheel_Joint
- removed joint FrontLeft_Wheel_Joint
- removed joint FrontRight_Wheel_Joint
- added joint left_back_wheel_joint: type continuous, parent base_link, child left_back_wheel_link, origin xyz=0.1375 -0.1 -0.01 rpy=0 0 0, axis 0 1 0, limit effort=100 velocity=100
- added joint left_front_wheel_joint: type continuous, parent base_link, child left_front_wheel_link, origin xyz=-0.1375 -0.1 -0.01 rpy=0 0 0, axis 0 1 0, limit effort=100 velocity=100
- added joint right_back_wheel_joint: type continuous, parent base_link, child right_back_wheel_link, origin xyz=0.1375 0.1 -0.01 rpy=3.1416 0 0, axis 0 1 0, limit effort=100 velocity=100
- added joint right_front_wheel_joint: type continuous, parent base_link, child right_front_wheel_link, origin xyz=-0.1375 0.1 -0.01 rpy=3.1416 0 0, axis 0 1 0, limit effort=100 velocity=100
